File: pcb/kicad/ToothEater/ToothEater.kicad_pcb (KiCad board)
At the start: 2 copper layers, 44 x 44 mm, 33 parts, among them J1 Conn_02x02_Molex, J2 Conn_02x02_Molex, Q1 BD681, Q2 BC546, Q3 BC546, Q4 BC546, Q5 BC546, Q6 BC546, U1 ATTINY85-20PU-ND, U2 VR_Conditioner_8-Pin-DIP, U3 MCP100

Commit message: - PCB v1.1 preparation.
Parts:
- removed D6: LED_3.3mm, LED_THT:LED_D3.0mm_IRBlack
- added TP1: TestPoint, TestPoint:TestPoint_Pad_1.0x1.0mm, F.Cu at (120.7, 73.2)
- R11: value 1k -> 4k7
- R3, R5: value 1k -> 10k
- R4, R6: value 10k -> 1k
- R7, R9: value 1k -> 47k
- moved Q6 10.5 mm to (124.7, 62.1), turned to 180 degrees
- moved R12 10.4 mm to (128.0, 70.6), turned to 0 degrees
- moved R11 8.81 mm to (122.8, 70.6), turned to 0 degrees
- moved U3 4.24 mm to (122.5, 90.7), turned to 90 degrees
- moved R7 1.23 mm to (122.8, 67.3)
- moved R8 1.21 mm to (130.0, 67.3)
Connections:
- net PB3_TEST_OUT renamed PB3_TACHO_OUT
- D1 pad 1: Net-(D1-Pad1) -> 12v_SAFE
- D4 pad 1: GND -> Net-(D4-Pad1)
- D5 pad 1: GND -> Net-(D5-Pad1)
- J2 pad 1: unconnected-(J2-Pad1) -> TACHO_OUT_PAD
- Q1 pad 2: Net-(D1-Pad1) -> 12v_SAFE
- Q4 pad 1: +5.2V_REG -> Net-(D4-Pad1)
- Q4 pad 3: Net-(Q4-Pad3) -> GND
- Q5 pad 1: +5.2V_REG -> Net-(D5-Pad1)
- Q5 pad 3: Net-(Q5-Pad3) -> GND
- Q6 pad 1: +5.2V_REG -> TACHO_OUT_PAD
- Q6 pad 3: Net-(Q6-Pad3) -> GND
- R1 pad 1: Net-(D1-Pad1) -> 12v_SAFE
- R10 pad 1: Net-(Q5-Pad3) -> +5.2V_REG
- R12 pad 1: Net-(Q6-Pad3) -> 12v_SAFE
- R12 pad 2: Net-(D6-Pad2) -> TACHO_OUT_PAD
- R8 pad 1: Net-(Q4-Pad3) -> +5.2V_REG
Routing:
- net 12v_SAFE: track 0.00 -> 57.0 mm, vias 0 -> 3
- net TACHO_OUT_PAD: track 0.00 -> 46.0 mm
- net Net-(Q4-Pad3): track 19.2 -> 0.00 mm
- net Net-(D1-Pad1): track 19.1 -> 0.00 mm
- net Net-(Q6-Pad3): track 16.2 -> 0.00 mm
- net PB3_TACHO_OUT: track 26.0 -> 11.5 mm
- net Net-(D5-Pad1): track 0.00 -> 11.0 mm
- net Net-(D4-Pad1): track 0.00 -> 9.69 mm
- net Net-(D6-Pad2): track 8.49 -> 0.00 mm
- net +5.2V_REG: track 132.7 -> 124.3 mm
- net VR_TTL_CRANK_OUT: track 44.0 -> 51.8 mm
- net Net-(Q5-Pad3): track 7.54 -> 0.00 mm
- net GND: track 24.7 -> 20.9 mm, vias 7 -> 5
- net PB4_CRANK_ENABLE_OUT: track 44.1 -> 41.0 mm
- net PB0_CAM_ENABLE_OUT: track 35.3 -> 33.3 mm
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Other:
- board text added: "TACHO"
- board text added: "Tooth Eater Module - v1.1 - Through-hole version Licensed under the CERN-OHL-S © 2026 Alex Kiaos"
- board text removed: "TEST"
- board text removed: "Tooth Eater Module - v1.0 - Through-hole version Licensed under the CERN-OHL-S © 2026 Alex Kiaos"
