File: pcb/kicad/ToothEater/ToothEater.kicad_pcb (KiCad board)
At the start: 2 copper layers, 44 x 44 mm, 33 parts, among them J1 Conn_02x02_Molex, J2 Conn_02x02_Molex, Q1 BD681, Q2 BC546, Q3 BC546, Q4 BC546, Q5 BC546, Q6 BC546, U1 ATTINY85-20PU-ND, U2 VR_Conditioner_8-Pin-DIP, U3 MCP100

Commit message: - PCB v1.1 preparation.
Routing:
- net VR_TTL_CRANK_OUT: track 51.8 -> 60.4 mm
- net GND: track 20.9 -> 27.0 mm, vias 5 -> 7
Changed lines of the file:
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@@
     (property "Sheetname" "")
     (attr through_hole)
-    (fp_text reference "R8" (at 3.302 2.032) (layer "F.SilkS")
+    (fp_text reference "R8" (at 3.302 1.778) (layer "F.SilkS")
       (effects (font (size 0.7 0.7) (thickness 0.15)))
     )
@@
     (property "Sheetname" "")
     (attr through_hole)
-    (fp_text reference "R7" (at -0.84 -1.778) (layer "F.SilkS")
+    (fp_text reference "R7" (at -1.348 -1.524) (layer "F.SilkS")
       (effects (font (size 0.7 0.7) (thickness 0.15)))
     )
@@
     (property "Sheetname" "")
     (attr through_hole)
-    (fp_text reference "D4" (at -0.757 2.286) (layer "F.SilkS")
+    (fp_text reference "D4" (at -0.249 2.54) (layer "F.SilkS")
       (effects (font (size 1 1) (thickness 0.15)))
     )
@@
   (segment (start 157.226 71.374) (end 157.226 74.676) (width 1) (layer "F.Cu") (net 1))
   (segment (start 131.064 89.916) (end 131.064 88.9) (width 1) (layer "F.Cu") (net 1))
+  (segment (start 136.652 88.9) (end 136.652 82.804) (width 0.8) (layer "F.Cu") (net 1))
   (segment (start 146.812 89.154) (end 146.558 89.408) (width 1) (layer "F.Cu") (net 1))
   (segment (start 131.064 88.9) (end 128.524 86.36) (width 1) (layer "F.Cu") (net 1))
   (via (at 146.558 89.408) (size 0.8) (drill 0.4) (layers "F.Cu" "B.Cu") (free) (net 1))
+  (via (at 136.652 82.804) (size 0.8) (drill 0.4) (layers "F.Cu" "B.Cu") (free) (net 1))
+  (via (at 136.652 88.9) (size 0.8) (drill 0.4) (layers "F.Cu" "B.Cu") (free) (net 1))
   (via (at 159.766 77.216) (size 0.8) (drill 0.4) (layers "F.Cu" "B.Cu") (free) (net 1))
   (via (at 131.064 89.916) (size 0.8) (drill 0.4) (layers "F.Cu" "B.Cu") (free) (net 1))
@@
   (segment (start 144.384 86.472) (end 141.234 83.322) (width 0.4) (layer "B.Cu") (net 14))
   (segment (start 145.917 86.472) (end 145.034 86.472) (width 0.4) (layer "B.Cu") (net 14))
-  (segment (start 142.494 89.916) (end 143.256 89.154) (width 0.4) (layer "F.Cu") (net 15))
-  (segment (start 143.256 89.154) (end 143.256 84.582) (width 0.4) (layer "F.Cu") (net 15))
-  (segment (start 139.446 89.916) (end 142.494 89.916) (width 0.4) (layer "F.Cu") (net 15))
-  (segment (start 137.932 88.402) (end 139.446 89.916) (width 0.4) (layer "F.Cu") (net 15))
+  (segment (start 146.304 79.756) (end 145.288 78.74) (width 0.4) (layer "F.Cu") (net 15))
   (segment (start 153.924 84.582) (end 155.448 83.058) (width 0.4) (layer "F.Cu") (net 15))
   (segment (start 132.598 88.402) (end 133.614 88.402) (width 0.4) (layer "F.Cu") (net 15))
   (segment (start 129.804 81.29) (end 131.572 83.058) (width 0.4) (layer "F.Cu") (net 15))
+  (segment (start 136.652 78.74) (end 135.382 80.01) (width 0.4) (layer "F.Cu") (net 15))
   (segment (start 131.572 87.376) (end 132.598 88.402) (width 0.4) (layer "F.Cu") (net 15))
+  (segment (start 135.382 87.63) (end 134.61 88.402) (width 0.4) (layer "F.Cu") (net 15))
   (segment (start 144.78 83.058) (end 146.304 84.582) (width 0.4) (layer "F.Cu") (net 15))
   (segment (start 146.304 84.582) (end 153.924 84.582) (width 0.4) (layer "F.Cu") (net 15))
   (segment (start 129.296 81.29) (end 129.804 81.29) (width 0.4) (layer "F.Cu") (net 15))
+  (segment (start 145.542 83.058) (end 146.304 82.296) (width 0.4) (layer "F.Cu") (net 15))
   (segment (start 155.448 83.058) (end 155.448 74.168) (width 0.4) (layer "F.Cu") (net 15))
   (segment (start 153.162 73.152) (end 153.162 71.988) (width 0.4) (layer "F.Cu") (net 15))
-  (segment (start 133.614 88.402) (end 137.932 88.402) (width 0.4) (layer "F.Cu") (net 15))
   (segment (start 155.448 74.168) (end 154.94 73.66) (width 0.4) (layer "F.Cu") (net 15))
   (segment (start 131.572 83.058) (end 131.572 87.376) (width 0.4) (layer "F.Cu") (net 15))
-  (segment (start 143.256 84.582) (end 144.78 83.058) (width 0.4) (layer "F.Cu") (net 15))
   (segment (start 154.94 73.66) (end 153.67 73.66) (width 0.4) (layer "F.Cu") (net 15))
+  (segment (start 134.61 88.402) (end 133.614 88.402) (width 0.4) (layer "F.Cu") (net 15))
+  (segment (start 144.78 83.058) (end 145.542 83.058) (width 0.4) (layer "F.Cu") (net 15))
+  (segment (start 145.288 78.74) (end 136.652 78.74) (width 0.4) (layer "F.Cu") (net 15))
+  (segment (start 146.304 82.296) (end 146.304 79.756) (width 0.4) (layer "F.Cu") (net 15))
+  (segment (start 135.382 80.01) (end 135.382 87.63) (width 0.4) (layer "F.Cu") (net 15))
   (segment (start 153.67 73.66) (end 153.162 73.152) (width 0.4) (layer "F.Cu") (net 15))
   (via (at 144.78 83.058) (size 0.8) (drill 0.4) (layers "F.Cu" "B.Cu") (net 15))
