File: pcb/kicad/ToothEater/ToothEater.kicad_sch (KiCad schematic)
At the start: 33 parts, among them J1 Conn_02x02_Molex, J2 Conn_02x02_Molex, Q1 BD681, Q2 BC546, Q3 BC546, Q4 BC546, Q5 BC546, Q6 BC546, U1 ATTINY85-20PU-ND, U2 VR_Conditioner_8-Pin-DIP, U3 MCP100

Commit message: - PCB v1.1 preparation.
Parts:
- removed D6: LED_3.3mm, LED_THT:LED_D3.0mm_IRBlack, symbol ToothEater:LED_3.3mm
- added TP1: TestPoint, TestPoint:TestPoint_Pad_1.0x1.0mm, symbol Connector:TestPoint
- R11: value 1k -> 4k7
- R3, R5: value 1k -> 10k
- R4, R6: value 10k -> 1k
- R7, R9: value 1k -> 47k
Connections:
- net +5.2V_REG: now also R10.1, R8.1; no longer Q4.1 (C), Q5.1 (C), Q6.1 (C)
- net GND: now also Q4.3 (E), Q5.3 (E), Q6.3 (E); no longer D4.1 (K), D5.1 (K)
- net 12v_SAFE: now reaches R12.1
- net 12v_SAFE: now also D1.1 (K), Q1.2 (C), R1.1; no longer Q6.3 (E)
- net TACHO_OUT_PAD: now reaches J2.1 (Pin_1)
- net TACHO_OUT_PAD: now also Q6.1 (C), R12.2
- net PB3_TEST_OUT renamed PB3_TACHO_OUT
- net PB3_TACHO_OUT: now also TP1.1
- new net: D4.1 (K), Q4.1 (C)
- new net: D5.1 (K), Q5.1 (C)
Other:
- note added: "10K also ok for base resistor"
- note added: "Approx 0 to 4.1v output"
- note added: "CRANK and CAM OUTPUTS"
- note added: "Cam Output Enable line to ECU. Post tooth filtering output only, (under firmware control). (Approx 0 to 4.16v output)"
- note added: "Crank Output line to ECU. Pass-through of VR Crank signal, (under firmware control). (Approx 0 to 4.16v output)"
- note added: "July 2026"
- note added: "TACHO"
- note added: "Test LEDS (Optional Installation)"
- note added: "Tooth-Eater Module (v1.1) POWER, VR socket, Micro & Leds"
- note removed: "Cam Output Enable line to ECU. Post tooth filtering output only, (under firmware control)."
- note removed: "Crank Output line to ECU. Pass-through of VR Crank signal, (under firmware control)."
- note removed: "May 2026"
- note removed: "Test LEDS - (Optional Installation)"
- note removed: "Through-hole version (v1.0)"
- note removed: "Tooth-Eater Module (v1.0) POWER, VR socket, Micro & Leds"
- moved on the sheet: D4, D5, JP1, JP2, Q2, Q3, Q4, Q5, R10, R3, R4, R5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
